Commit message: move on start_LED

File: src/grr_description/bloodstone.urdf (robot description, URDF)
Before this commit: robot bloodstone, 53 links, 52 joints
Links:
- link camera_1_link: geometry collision box size=0.575 0.016 0.25; visual mesh filename=package://grr_description/meshes/camera.stl scale=0.001 0.001 0.001
- link camera_2_link: geometry collision box size=0.575 0.016 0.25; visual mesh filename=package://grr_description/meshes/camera.stl scale=0.001 0.001 0.001
