Commit message: add joint_trarjectory controller and odom set function

File: src/grr_description/urdf/control/drive.xacro (robot description, xacro)
@@ -39,4 +39,14 @@
       <state_interface name="velocity"/>
     </joint>
+    <joint name="small_package_grabber_roller_1_joint">
+      <command_interface name="effort"/>
+      <state_interface name="position"/>
+      <state_interface name="velocity"/>
+    </joint>
+    <joint name="small_package_sweeper_roller_joint">
+      <command_interface name="effort"/>
+      <state_interface name="position"/>
+      <state_interface name="velocity"/>
+    </joint>
   </ros2_control>
 </robot>

Commit message: effort controller added

File: src/grr_description/urdf/control/drive.xacro (robot description, xacro)
@@ -40,10 +40,10 @@
     </joint>
     <joint name="small_package_grabber_roller_1_joint">
-      <command_interface name="velocity"/>
+      <command_interface name="effort"/>
       <state_interface name="position"/>
       <state_interface name="velocity"/>
     </joint>
     <joint name="small_package_sweeper_roller_joint">
-      <command_interface name="velocity"/>
+      <command_interface name="effort"/>
       <state_interface name="position"/>
       <state_interface name="velocity"/>

File: src/grr_description/urdf/parts/small_package_sweeper.xacro (robot description, xacro)
@@ -85,5 +85,5 @@
       <child link="small_package_sweeper_link"/>
       <axis xyz="1 0 0"/>
-      <limit effort="100" lower="-1.57" upper="1.57" velocity="0.5"/>
+      <limit effort="100" lower="-1.57" upper="1.57" velocity="10"/>
     </joint>
     <link name="small_package_sweeper_roller_link">
